File: servo-shield.brd (EAGLE design)
At the start: 65 x 56 mm, 30 parts, among them IC1 24AA01P, K1 PIN20X2

Commit message: So bored. Curves. still passes DRC.
Parts:
- moved C4 40.3 mm to (17.9, 3.02), turned to 0 degrees
- moved RN2 0.50 mm to (20.7, 16.0)
Routing:
- net +3V3: track 154.3 -> 110.5 mm
- net ID_SCL: track 74.1 -> 61.0 mm
- net ID_SDA: track 64.4 -> 52.2 mm
- net I2C_SDA: track 91.4 -> 80.7 mm
- net I2C_SCL: track 87.0 -> 76.5 mm
- net +5V: track 89.6 -> 80.0 mm
- net V+: track 113.5 -> 107.2 mm
- net N$23: track 25.7 -> 20.6 mm
- net N$24: track 22.5 -> 17.6 mm
- net N$25: track 19.3 -> 14.6 mm
- net N$34: track 23.2 -> 18.8 mm
- net N$35: track 26.4 -> 22.0 mm
- net N$33: track 20.1 -> 15.7 mm
- net N$26: track 16.1 -> 11.8 mm
- net N$32: track 16.9 -> 12.6 mm
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